Commit message: Added Isaac Sim support

File: onrobot_rg_description/urdf/onrobot_rg2_model_macro.xacro (robot description, xacro)
@@ -24,4 +24,5 @@
           <mesh filename="package://onrobot_rg_description/meshes/rg2/collision/outer_knuckle.stl" />
         </geometry>
+        <sdf resolution="512"/>
       </collision>
     </link>
@@ -54,4 +55,5 @@
           <mesh filename="package://onrobot_rg_description/meshes/rg2/collision/inner_knuckle.stl" />
         </geometry>
+        <sdf resolution="512"/>
       </collision>
     </link>
@@ -84,4 +86,5 @@
           <mesh filename="package://onrobot_rg_description/meshes/rg2/collision/inner_finger.stl" />
         </geometry>
+        <sdf resolution="512"/>
       </collision>
     </link>

File: onrobot_rg_description/urdf/onrobot_rg6.xacro (robot description, xacro)
@@ -1,5 +1,5 @@
 <?xml version="1.0"?>
 <robot xmlns:xacro="http://ros.org/wiki/xacro">
-  <xacro:macro name="base_link" params="prefix effector_base:=world">
+  <xacro:macro name="base_link" params="prefix">
     <link name="${prefix}base_link">
       <inertial>
@@ -24,13 +24,4 @@
       </collision>
     </link>
-    <xacro:property name="generate_world" value="${effector_base == 'world'}"/>
-    <xacro:if value="${generate_world}">
-      <link name="world"/>
-    </xacro:if>
-    <joint name="joint0" type="fixed">
-        <parent link="${effector_base}"/>
-        <child link="${prefix}base_link"/>
-        <origin xyz= "0. 0. 0." rpy="0. 0. 1.57" />
-    </joint>
     <gazebo reference="${prefix}base_link">
       <mu1>1.0</mu1>

File: onrobot_rg_description/urdf/onrobot_rg6_model_macro.xacro (robot description, xacro)
@@ -138,6 +138,6 @@
     <xacro:finger_joints prefix="${prefix}" fingerprefix="right" reflect="-1.0"/>
   </xacro:macro>
-  <xacro:macro name="onrobot_rg6" params="prefix effector_base:=world">
-    <xacro:base_link prefix="${prefix}" effector_base="${effector_base}"/>
+  <xacro:macro name="onrobot_rg6" params="prefix">
+    <xacro:base_link prefix="${prefix}"/>
     <xacro:finger_links prefix="${prefix}" fingerprefix="left"/>
     <xacro:finger_links prefix="${prefix}" fingerprefix="right"/>
