Commit message: Reworked whole communication physical device & Isaac Sim works, simulated WIP.

File: onrobot_rg_description/urdf/onrobot_rg6_gazebo.xacro (robot description, xacro)
@@ -9,7 +9,23 @@
     </gazebo>
     <gazebo>
-      <plugin filename="libroboticsgroup_upatras_gazebo_mimic_joint_plugin.so" name="mimic_${prefix}left_inner_knuckle_joint">
-        <joint>${prefix}finger_joint</joint>
-        <mimicJoint>${prefix}left_inner_knuckle_joint</mimicJoint>
+      <plugin filename="libroboticsgroup_upatras_gazebo_mimic_joint_plugin.so" name="mimic_left_inner_knuckle_joint">
+        <joint>finger_joint</joint>
+        <mimicJoint>left_inner_knuckle_joint</mimicJoint>
+        <multiplier>1.0</multiplier>
+        <offset>0.0</offset>
+        <maxEffort>5.0</maxEffort>
+        <!-- <hasPID /> -->
+      </plugin>
+      <plugin filename="libroboticsgroup_upatras_gazebo_mimic_joint_plugin.so" name="mimic_right_inner_knuckle_joint">
+        <joint>finger_joint</joint>
+        <mimicJoint>right_inner_knuckle_joint</mimicJoint>
+        <multiplier>1.0</multiplier>
+        <offset>0.0</offset>
+        <maxEffort>5.0</maxEffort>
+        <!-- <hasPID /> -->
+      </plugin>
+      <plugin filename="libroboticsgroup_upatras_gazebo_mimic_joint_plugin.so" name="mimic_left_inner_finger_joint">
+        <joint>finger_joint</joint>
+        <mimicJoint>left_inner_finger_joint</mimicJoint>
         <multiplier>-1.0</multiplier>
         <offset>0.0</offset>
@@ -17,7 +33,7 @@
         <!-- <hasPID /> -->
       </plugin>
-      <plugin filename="libroboticsgroup_upatras_gazebo_mimic_joint_plugin.so" name="mimic_${prefix}right_inner_knuckle_joint">
-        <joint>${prefix}finger_joint</joint>
-        <mimicJoint>${prefix}right_inner_knuckle_joint</mimicJoint>
+      <plugin filename="libroboticsgroup_upatras_gazebo_mimic_joint_plugin.so" name="mimic_right_inner_finger_joint">
+        <joint>finger_joint</joint>
+        <mimicJoint>right_inner_finger_joint</mimicJoint>
         <multiplier>-1.0</multiplier>
         <offset>0.0</offset>
@@ -25,24 +41,8 @@
         <!-- <hasPID /> -->
       </plugin>
-      <plugin filename="libroboticsgroup_upatras_gazebo_mimic_joint_plugin.so" name="mimic_${prefix}left_inner_finger_joint">
-        <joint>${prefix}finger_joint</joint>
-        <mimicJoint>${prefix}left_inner_finger_joint</mimicJoint>
+      <plugin filename="libroboticsgroup_upatras_gazebo_mimic_joint_plugin.so" name="mimic_right_outer_knuckle_joint">
+        <joint>finger_joint</joint>
+        <mimicJoint>right_outer_knuckle_joint</mimicJoint>
         <multiplier>1.0</multiplier>
-        <offset>0.0</offset>
-        <maxEffort>5.0</maxEffort>
-        <!-- <hasPID /> -->
-      </plugin>
-      <plugin filename="libroboticsgroup_upatras_gazebo_mimic_joint_plugin.so" name="mimic_${prefix}right_inner_finger_joint">
-        <joint>${prefix}finger_joint</joint>
-        <mimicJoint>${prefix}right_inner_finger_joint</mimicJoint>
-        <multiplier>1.0</multiplier>
-        <offset>0.0</offset>
-        <maxEffort>5.0</maxEffort>
-        <!-- <hasPID /> -->
-      </plugin>
-      <plugin filename="libroboticsgroup_upatras_gazebo_mimic_joint_plugin.so" name="mimic_${prefix}right_outer_knuckle_joint">
-        <joint>${prefix}finger_joint</joint>
-        <mimicJoint>${prefix}right_outer_knuckle_joint</mimicJoint>
-        <multiplier>-1.0</multiplier>
         <offset>0.0</offset>
         <maxEffort>5.0</maxEffort>
